Commit message: fix: SLAM scan matching failure - camera optical frame rotation & odometry fallback
3 root causes fixed:

1. Camera optical frame mismatch: Gazebo depth cameras output points in
   optical convention (Z=forward, X=right, Y=down) but makeCameraTransform()
   assumed ROS base convention (X=forward, Y=left, Z=up). Added rotation
   matrix to convert optical→base frame before applying camera pose.
   This caused fitness scores ~25.77 (should be <1.0).

2. Map not growing: When scan matching failed, no keyframes were added.
   Now odometry fallback still adds keyframes and raycasts to OctoMap,
   so the map keeps growing even without scan matching convergence.

3. URDF: Added camera_link parent frame grouping all 4 cameras under
   a single TF parent instead of directly on base_link.

Also tuned GICP params: max_corr_dist 1.0→2.0, fitness_threshold 0.5→1.0,
max_iterations 50→64, self_filter_size 0.6→0.5.

https://claude.ai/code/session_016hU2xQwzMfVdEDm5cveysb

File: src/agv_sim/urdf/agv.urdf.xacro (robot description, xacro)
@@ -46,4 +46,11 @@
   <xacro:caster name="front_caster" x="0.3"/>
   <xacro:caster name="rear_caster" x="-0.3"/>
+  <!-- Parent frame untuk semua kamera -->
+  <link name="camera_link"/>
+  <joint name="camera_joint" type="fixed">
+    <parent link="base_link"/>
+    <child link="camera_link"/>
+    <origin xyz="0 0 0" rpy="0 0 0"/>
+  </joint>
   <xacro:macro name="kinect_v1" params="name x y yaw topic">
     <link name="${name}_link">
@@ -51,5 +58,5 @@
     </link>
     <joint name="${name}_joint" type="fixed">
-      <parent link="base_link"/><child link="${name}_link"/><origin xyz="${x} ${y} 0.4" rpy="0 0 ${yaw}"/>
+      <parent link="camera_link"/><child link="${name}_link"/><origin xyz="${x} ${y} 0.4" rpy="0 0 ${yaw}"/>
     </joint>
     <gazebo reference="${name}_link">

Commit message: feat: rewrite SLAM with scan-to-submap matching (lidarslam_ros2 approach)
Complete rewrite of the SLAM system:

1. URDF: Added optical frames for each camera. Gazebo depth cameras
   output points in optical convention (Z=forward,X=right,Y=down).
   The optical frame link + TF2 properly converts to base_link.
   Camera hierarchy: base_link → camera_link → camera_link_N_link → camera_link_N_optical

2. SLAM Node: Replaced custom GICP+OctoMap with scan-to-submap matching
   based on lidarslam_ros2 architecture:
   - Subscribes to /full_pointcloud (merged by pointcloud_concatenate)
   - Uses odometry as initial guess via TF2 odom→base_link lookup
   - GICP/NDT alignment against targeted_cloud (N recent submaps)
   - Background thread for map updates
   - Publishes map→odom TF, map cloud, trajectory, pose
   - Removed OctoMap dependency, removed manual camera merging

3. Launch: Added pointcloud_concatenate node to pipeline:
   Gazebo → 4x cameras → pointcloud_concatenate (TF2) → SLAM node
   This separates camera fusion from SLAM logic cleanly.

4. Config: New parameters matching lidarslam_ros2 style
   (registration_method, trans_for_mapupdate, num_targeted_cloud, etc.)

https://claude.ai/code/session_016hU2xQwzMfVdEDm5cveysb

File: src/agv_sim/urdf/agv.urdf.xacro (robot description, xacro)
@@ -53,5 +53,12 @@
     <origin xyz="0 0 0" rpy="0 0 0"/>
   </joint>
+  <!--
+    Macro kamera RGBD dengan optical frame.
+    Gazebo depth camera menghasilkan point cloud dalam optical frame convention
+    (Z=forward/depth, X=right, Y=down). Optical frame link ditambahkan agar
+    TF2 bisa transformasi langsung ke base_link dengan benar.
+  -->
   <xacro:macro name="kinect_v1" params="name x y yaw topic">
+    <!-- Link fisik kamera -->
     <link name="${name}_link">
       <visual><geometry><box size="0.05 0.12 0.04"/></geometry><material name="blue"><color rgba="0 0 0.8 1"/></material></visual>
@@ -60,9 +67,17 @@
       <parent link="camera_link"/><child link="${name}_link"/><origin xyz="${x} ${y} 0.4" rpy="0 0 ${yaw}"/>
     </joint>
+    <!-- Optical frame: rotasi dari link frame (x-forward,y-left,z-up) ke optical (z-forward,x-right,y-down) -->
+    <link name="${name}_optical"/>
+    <joint name="${name}_optical_joint" type="fixed">
+      <parent link="${name}_link"/>
+      <child link="${name}_optical"/>
+      <origin xyz="0 0 0" rpy="${-pi/2} 0 ${-pi/2}"/>
+    </joint>
     <gazebo reference="${name}_link">
       <sensor name="${name}" type="depth_camera">
         <update_rate>20</update_rate>
         <topic>${topic}</topic>
-        <gz_frame_id>${name}_link</gz_frame_id>
+        <!-- Publish point cloud dalam optical frame agar TF2 bisa transform ke base_link -->
+        <gz_frame_id>${name}_optical</gz_frame_id>
         <camera><horizontal_fov>1.047</horizontal_fov><image><width>640</width><height>480</height></image><clip><near>0.5</near><far>8.0</far></clip></camera>
       </sensor>
